Commit message: navigation problem solved.yay

File: urdf/lidar.xacro (robot description, xacro)
@@ -5,5 +5,5 @@
     <xacro:property name="camera_height" value="0.05" />
     <!--camera link-->
-    <link name="lidar_link">
+    <link name="base_scan">
         <visual>
             <geometry>
@@ -20,10 +20,10 @@
                             xyz="0 0 0" rpy="0 1.57 0" />
     </link>
-    <joint name="head_lidar_joint" type="fixed">
+    <!-- <joint name="head_lidar_joint" type="fixed">
         <parent link="head_link"/>
         <child link="lidar_link"/>
         <origin xyz="0 0 ${head_radius}" rpy="0 0 0"/>
-    </joint>
-    <gazebo reference="lidar_link">
+    </joint> -->
+    <gazebo reference="base_scan">
         <sensor type="ray" name="lidar_sensor">
             <pose>0 0 0 0 0 0</pose>
@@ -45,6 +45,10 @@
             </ray>
             <plugin name="turtlebot3_laserscan" filename="libgazebo_ros_ray_sensor.so">
+                <ros>
+                    <remapping>/turtlebot3_laserscan/out:=/scan</remapping>
+                </ros>
                 <output_type>sensor_msgs/LaserScan</output_type>
-                <frame_name>lidar_link</frame_name>
+                <frame_name>base_scan</frame_name>
+                <topic>/scan</topic>
             </plugin>
         </sensor>

File: urdf/medibot.urdf (robot description, URDF)
Before this commit: robot medibot, 15 links, 14 joints
Links:
- removed link lidar_link
- added link base_scan, mass 0.1; collision box size=0.01 0.1 0.05; visual box size=0.01 0.1 0.05
Joints:
- removed joint base_upper_joint
- removed joint head_lidar_joint
- added joint base_lider_joint: type fixed, parent base_link, child base_scan, origin xyz=0.06 0 0.225 rpy=0 0 0
- added joint lider_upper_joint: type fixed, parent base_scan, child body_base_link, origin xyz=0.06 0 0.25 rpy=0 0 0
- joint body_shoulder_joint: type revolute -> fixed

File: urdf/medibot.urdf.xacro (robot description, xacro)
@@ -9,8 +9,13 @@
     <xacro:include filename="lidar.xacro" />
     <xacro:include filename="imu.xacro" />
-    <joint name="base_upper_joint" type="fixed">
+    <joint name="base_lider_joint" type="fixed">
         <parent link="base_link" />
+        <child link="base_scan" />
+        <origin xyz="${base_length/10} 0 ${base_height+camera_height/2}" rpy="0 0 0"/>
+    </joint>
+    <joint name="lider_upper_joint" type="fixed">
+        <parent link="base_scan" />
         <child link="body_base_link" />
-        <origin xyz="${base_length/10} 0 ${base_height+body_length/2}" rpy="0 0 0"/>
+        <origin xyz="${base_length/10} 0 ${base_height+camera_height}" rpy="0 0 0"/>
     </joint>
 </robot>

File: urdf/mobile_base_gazebo.xacro (robot description, xacro)
@@ -25,13 +25,9 @@
     <gazebo>
         <plugin name="diff_drive_controller" filename="libgazebo_ros_diff_drive.so">
-            <!-- Update rate in Hz -->
             <update_rate>50</update_rate>
-            <!-- wheels -->
             <left_joint>wheel_left_joint</left_joint>
             <right_joint>wheel_right_joint</right_joint>
-            <!-- kinematics -->
             <wheel_separation>0.45</wheel_separation>
             <wheel_diameter>0.2</wheel_diameter>
-            <!-- output -->
             <publish_odom>true</publish_odom>
             <publish_odom_tf>true</publish_odom_tf>
@@ -39,5 +35,5 @@
             <odometry_topic>odom</odometry_topic>
             <odometry_frame>odom</odometry_frame>
-            <robot_base_frame>base_link</robot_base_frame>
+            <robot_base_frame>base_footprint</robot_base_frame>
         </plugin>
     </gazebo>

File: urdf/upper_base.urdf.xacro (robot description, xacro)
@@ -136,5 +136,5 @@
                             xyz="0 0 0" rpy="0 0 0" />
     </link>
-    <joint name="body_shoulder_joint" type="revolute">
+    <joint name="body_shoulder_joint" type="fixed">
         <parent link="body_base_link"/>
         <child link="shoulder_link"/>
