Commit message: baymax added

File: urdf/camera_gazebo.xacro (robot description, xacro)
@@ -1,7 +1,4 @@
 <?xml version="1.0"?>
 <robot name="medibot" xmlns:xacro="http://www.ros.org/wiki/xacro">
-    <xacro:property name="camera_length" value="0.01" />
-    <xacro:property name="camera_width" value="0.1" />
-    <xacro:property name="camera_height" value="0.05" />
     <!--camera link-->
     <link name="camera_link">
@@ -20,9 +17,9 @@
                             xyz="0 0 0" rpy="0 0 0" />
     </link>
-    <joint name="head_camera_joint" type="fixed">
+    <!-- <joint name="head_camera_joint" type="fixed">
         <parent link="head_link"/>
         <child link="camera_link"/>
         <origin xyz="${head_radius} 0 0" rpy="0 0 0"/>
-    </joint>
+    </joint> -->
     <gazebo reference="camera_link">
         <material>

File: urdf/common_properties.xacro (robot description, xacro)
@@ -1,4 +1,20 @@
 <?xml version="1.0"?>
 <robot xmlns:xacro="http://www.ros.org/wiki/xacro">
+    <xacro:property name="base_length" value="0.6" />
+    <xacro:property name="base_width" value="0.4" />
+    <xacro:property name="base_height" value="0.2" />
+    <xacro:property name="wheel_radius" value="0.1" />
+    <xacro:property name="wheel_length" value="0.05" />
+    <xacro:property name="body_length" value="0.5" />
+    <xacro:property name="body_radius" value="0.1" />
+    <xacro:property name="shoulder_length" value="0.1" />
+    <xacro:property name="shoulder_width" value="0.4" />
+    <xacro:property name="shoulder_height" value="0.2" />
+    <xacro:property name="hand_height" value="0.2" />
+    <xacro:property name="hand_radius" value="0.05" />
+    <xacro:property name="head_radius" value="0.1" />
+    <xacro:property name="camera_length" value="0.01" />
+    <xacro:property name="camera_width" value="0.1" />
+    <xacro:property name="camera_height" value="0.05" />
     <material name="blue">
         <color rgba="0 0 0.5 1" />

File: urdf/imu.xacro (robot description, xacro)
@@ -23,5 +23,5 @@
         <parent link="base_link"/>
         <child link="imu_link"/>
-        <origin xyz="${base_length/2-0.1} 0 ${base_height}" rpy="0 1.57 0"/>
+        <origin xyz="${base_length/2-camera_width} 0 ${base_height}" rpy="0 1.57 0"/>
     </joint>
     <gazebo reference="imu_link">
@@ -32,5 +32,5 @@
             <plugin name="my_imu_plugin" filename="libgazebo_ros_imu_sensor.so">
                 <ros>
-                <remapping>~/out:=imu</remapping>
+                    <remapping>~/out:=imu</remapping>
                 </ros>
             </plugin>

File: urdf/medibot.urdf (robot description, URDF)
Before this commit: robot medibot, 15 links, 14 joints
Links:
- removed link body_base_link
- removed link head_link
- removed link left_arm_link
- removed link left_hand_link
- removed link right_arm_link
- removed link right_hand_link
- removed link shoulder_link
- added link baymax_link, mass 1.0; collision mesh filename=file:///home/nabil/ros2_ws/src/medibot/urdf/Baymax.STL scale=0.007 0.007 0.007; visual mesh filename=file:///home/nabil/ros2_ws/src/medibot/urdf/Baymax.STL scale=0.007 0.007 0.007
Joints:
- removed joint body_shoulder_joint
- removed joint head_camera_joint
- removed joint left_hand_arm_joint
- removed joint left_hand_shoulder_joint
- removed joint lider_upper_joint
- removed joint right_hand_arm_joint
- removed joint right_hand_shoulder_joint
- removed joint shoulder_head_joint
- added joint baymax_camera_joint: type fixed, parent baymax_link, child camera_link, origin xyz=0.05 0 0.8 rpy=0 0 0
- added joint lider_baymax_joint: type fixed, parent base_scan, child baymax_link, origin xyz=0.06 0 0.25 rpy=0 0 0

File: urdf/mobile_base.xacro (robot description, xacro)
@@ -1,9 +1,9 @@
 <?xml version="1.0"?>
 <robot name="medibot" xmlns:xacro="http://www.ros.org/wiki/xacro">
-    <xacro:property name="base_length" value="0.6" />
+    <!-- <xacro:property name="base_length" value="0.6" />
     <xacro:property name="base_width" value="0.4" />
     <xacro:property name="base_height" value="0.2" />
     <xacro:property name="wheel_radius" value="0.1" />
-    <xacro:property name="wheel_length" value="0.05" />
+    <xacro:property name="wheel_length" value="0.05" /> -->
     <link name="base_footprint" />
     <link name="base_link">

File: urdf/old.xacro (robot description, xacro)
@@ -2,7 +2,6 @@
 <robot name="medibot" xmlns:xacro="http://www.ros.org/wiki/xacro">
     <xacro:include filename="common_properties.xacro" />
-    <!-- <xacro:include filename="upper_base.urdf.xacro" /> -->
-    <!-- <xacro:include filename="upper_base_gazebo.xacro" /> -->
-    <xacro:include filename="baymax.urdf.xacro" />
+    <xacro:include filename="upper_base.urdf.xacro" />
+    <xacro:include filename="upper_base_gazebo.xacro" />
     <xacro:include filename="mobile_base.xacro" />
     <xacro:include filename="mobile_base_gazebo.xacro" />
@@ -10,4 +9,9 @@
     <xacro:include filename="lidar.xacro" />
     <xacro:include filename="imu.xacro" />
+    <joint name="head_camera_joint" type="fixed">
+        <parent link="head_link"/>
+        <child link="camera_link"/>
+        <origin xyz="${head_radius} 0 0" rpy="0 0 0"/>
+    </joint>
     <joint name="base_lider_joint" type="fixed">
         <parent link="base_link" />
@@ -15,18 +19,8 @@
         <origin xyz="${base_length/10} 0 ${base_height+camera_height/2}" rpy="0 0 0"/>
     </joint>
-    <joint name="baymax_camera_joint" type="fixed">
-        <parent link="baymax_link"/>
-        <child link="camera_link"/>
-        <origin xyz="0.05 0 0.8" rpy="0 0 0"/>
-    </joint>
-    <!-- <joint name="lider_upper_joint" type="fixed">
+    <joint name="lider_upper_joint" type="fixed">
         <parent link="base_scan" />
         <child link="body_base_link" />
         <origin xyz="${base_length/10} 0 ${base_height+camera_height}" rpy="0 0 0"/>
-    </joint> -->
-    <joint name="lider_baymax_joint" type="fixed">
-        <parent link="base_scan" />
-        <child link="baymax_link" />
-        <origin xyz="${base_length/10} 0 ${base_height+camera_height}" rpy="0 0 0"/>
     </joint>
 </robot>

File: urdf/upper_base.urdf.xacro (robot description, xacro)
@@ -2,12 +2,12 @@
 <robot name="medibot" xmlns:xacro="http://www.ros.org/wiki/xacro">
     <!-- <xacro:include filename="common_properties.xacro" /> -->
-    <xacro:property name="body_length" value="0.5" />
+    <!-- <xacro:property name="body_length" value="0.5" />
     <xacro:property name="body_radius" value="0.1" />
     <xacro:property name="shoulder_length" value="0.1" />
-    <xacro:property name="shoulder_width" value="0.6" />
+    <xacro:property name="shoulder_width" value="0.4" />
     <xacro:property name="shoulder_height" value="0.2" />
-    <xacro:property name="hand_height" value="0.4" />
+    <xacro:property name="hand_height" value="0.2" />
     <xacro:property name="hand_radius" value="0.05" />
-    <xacro:property name="head_radius" value="0.1" />
+    <xacro:property name="head_radius" value="0.1" /> -->
     <!-- upper body link -->
     <link name="body_base_link">
@@ -86,5 +86,5 @@
         <visual>
             <geometry>
-                <cylinder radius="0.05" length="0.5"/>
+                <cylinder radius="${hand_radius}" length="${hand_height}"/>
             </geometry>
             <origin xyz="0 0 ${hand_height/2+head_radius/2}" rpy="0 0 0" />
@@ -93,5 +93,5 @@
         <collision>
             <geometry>
-                <cylinder radius="0.05" length="0.5"/>
+                <cylinder radius="${hand_radius}" length="${hand_height}"/>
             </geometry>
             <origin xyz="0 0 ${hand_height/2+head_radius/2}" rpy="0 0 0" />
@@ -122,5 +122,5 @@
         <visual>
             <geometry>
-                <cylinder radius="0.05" length="0.5"/>
+                <cylinder radius="${hand_radius}" length="${hand_height}"/>
             </geometry>
             <origin xyz="0 0 ${hand_height/2+head_radius/2}" rpy="0 0 0" />
@@ -129,5 +129,5 @@
         <collision>
             <geometry>
-                <cylinder radius="0.05" length="0.5"/>
+                <cylinder radius="${hand_radius}" length="${hand_height}"/>
             </geometry>
             <origin xyz="0 0 ${hand_height/2+head_radius/2}" rpy="0 0 0" />
